Commit message: Donut flying

File: conf/simulator/pybullet/coaxial_donut.urdf (robot description, URDF)
Before this commit: robot coaxial_donut, 5 links, 4 joints
Links:
- link mainbody: geometry collision box size=0.04 0.04 0.02; visual box size=0.1 0.05 0.02

Commit message: use measured inertia and mass

File: conf/simulator/pybullet/coaxial_donut.urdf (robot description, URDF)
Before this commit: robot coaxial_donut, 5 links, 4 joints
Links:
- link mainbody: mass 0.15 -> 0.9
